File: docs/circuit/go-kart_cockpit.kicad_pcb (KiCad board)
At the start: 2 copper layers, 105.2 x 57.2 mm, 33 parts, among them P1 Power, Q1 TIP120, X1 AVR-ISP-10, X10 Bluetooth-Modul, X11 Start/Stop/Rückwärts, X12 Taster rechts (male), X13 Taster links (male), X2 Display (male), X3 5V, X4 GND, X5 SDA, X6 24V Hupe, X7 J5, X8 J3, X9 SCL

Commit message: feat(circuit): final touches
Parts:
- removed JP10: Display_Vcc, Resistor_THT:R_Axial_DIN0207_L6.3mm_D2.5mm_P7.62mm_Horizontal
- removed JP12: Display_Vcc, Resistor_THT:R_Axial_DIN0207_L6.3mm_D2.5mm_P15.24mm_Horizontal
- removed JP3: ISP_SCK, Resistor_THT:R_Axial_DIN0207_L6.3mm_D2.5mm_P10.16mm_Horizontal
- removed JP4: ISP_MOSI, Resistor_THT:R_Axial_DIN0207_L6.3mm_D2.5mm_P15.24mm_Horizontal
- removed JP5: TXD0, Resistor_THT:R_Axial_DIN0207_L6.3mm_D2.5mm_P10.16mm_Horizontal
- removed JP6: RXD0, Resistor_THT:R_Axial_DIN0207_L6.3mm_D2.5mm_P10.16mm_Horizontal
- removed JP9: ~, Resistor_THT:R_Axial_DIN0207_L6.3mm_D2.5mm_P15.24mm_Horizontal
- added X12: PD7, Connector_PinSocket_2.54mm:PinSocket_1x01_P2.54mm_Vertical, F.Cu at (78.2, 84.2)
- added X14: PG4, Connector_PinSocket_2.54mm:PinSocket_1x01_P2.54mm_Vertical, F.Cu at (85.2, 78.5)
- added X6: CS, Connector_PinSocket_2.54mm:PinSocket_1x01_P2.54mm_Vertical, F.Cu at (91.5, 68.5)
- added X7: PB6, Connector_PinSocket_2.54mm:PinSocket_1x01_P2.54mm_Vertical, F.Cu at (81.2, 68.5)
- added XB10: ISP_SCK, Resistor_THT:R_Axial_DIN0207_L6.3mm_D2.5mm_P10.16mm_Horizontal, F.Cu at (132.7, 59.5)
- added XB2: ~, Resistor_THT:R_Axial_DIN0207_L6.3mm_D2.5mm_P15.24mm_Horizontal, F.Cu at (67.8, 100.4)
- added XB3: Display_Vcc, Resistor_THT:R_Axial_DIN0207_L6.3mm_D2.5mm_P7.62mm_Horizontal, F.Cu at (112.5, 81.0)
- added XB5: Display_Vcc, Resistor_THT:R_Axial_DIN0207_L6.3mm_D2.5mm_P15.24mm_Horizontal, F.Cu at (118.5, 73.5)
- added XB6: TXD0, Resistor_THT:R_Axial_DIN0207_L6.3mm_D2.5mm_P10.16mm_Horizontal, F.Cu at (113.2, 68.0)
- added XB7: RXD0, Resistor_THT:R_Axial_DIN0207_L6.3mm_D2.5mm_P10.16mm_Horizontal, F.Cu at (124.2, 68.0)
- added XB9: ISP_MOSI, Resistor_THT:R_Axial_DIN0207_L6.3mm_D2.5mm_P15.24mm_Horizontal, F.Cu at (143.0, 79.6)
- P1: moved to F.Cu
- XB4: renamed from JP8; value GND -> Display_GND
- moved R1 10.1 mm to (62.2, 58.8), turned to -90 degrees
- moved P1 3.55 mm to (57.8, 60.0), turned to -90 degrees
- moved X2 2.51 mm to (81.2, 73.0)
- moved X13 2.50 mm to (81.2, 78.5)
- moved X16 2.26 mm to (150.5, 62.4)
- moved XB8 1.75 mm to (129.2, 57.9)
- moved X17 1.73 mm to (154.2, 92.7)
- moved R10 1.50 mm to (143.5, 84.9)
- moved R9 1.27 mm to (148.2, 90.1)
- moved R8 0.90 mm to (138.2, 73.3)
- moved R5 0.46 mm to (108.0, 51.8)
- moved X3 0.25 mm to (67.5, 68.5)
- renumbered R2 to R1, R7 to R10, R3 to R4, R4 to R5, R5 to R6, R6 to R7, R1 to R8, R8 to R9, X12 to X1, X2 to X11, X5 to X13, X1 to X15, X13 to X16, X11 to X17, X3 to X2, X4 to X3, X6 to X4, X9 to X5, X7 to X8, X8 to X9, JP11 to XB1, JP2 to XB8
Connections:
- net Net-(X10-Pin_1) renamed /BL_RX3V3
- P1 pad 1: GND -> Net-(P1-K)
- P1 pad 2: Net-(P1-A) -> Vcc (5V)
- R1 pad 1: Vcc (5V) -> Net-(P1-K)
- R1 pad 2: Net-(P1-A) -> GND
- X11 pad 2: Net-(JP5-B) -> PE1_TXD0
- X11 pad 6: Net-(JP6-B) -> PE0_RXD0
- X15 pad 1: Net-(JP4-B) -> PB2_MOSI
- X15 pad 7: Net-(JP3-B) -> PB1_SCK
- X8 pad 11: unconnected-(X7-Pin_11-Pad11) -> /PG4
- X8 pad 17: unconnected-(X7-Pin_17-Pad17) -> /PD7
- X9 pad 12: unconnected-(X8-Pin_12-Pad12) -> /PB6_OC1B
- X9 pad 18: unconnected-(X8-Pin_18-Pad18) -> /PB0_CS
Routing:
- net PB2_MOSI: track 63.9 -> 92.8 mm
- net PE1_TXD0: track 17.4 -> 35.2 mm
- net PE0_RXD0: track 30.9 -> 45.4 mm
- net PB1_SCK: track 49.5 -> 63.4 mm
- net /PG4: track 0.00 -> 13.6 mm
- net Net-(JP4-B): track 12.9 -> 0.00 mm
- net Net-(JP6-B): track 8.68 -> 0.00 mm
- net Vcc (5V): track 228.1 -> 236.5 mm
- net Net-(JP5-B): track 7.62 -> 0.00 mm
- net /RESET: track 162.8 -> 155.7 mm
- net /PD7: track 0.00 -> 5.96 mm
- net /PB0_CS: track 0.00 -> 5.77 mm
- net Net-(JP3-B): track 5.42 -> 0.00 mm
- net Net-(P1-A): track 5.37 -> 0.00 mm
- net Net-(P1-K): track 0.00 -> 4.92 mm
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Other:
- board size 105.2 x 57.2 mm -> 103.5 x 57.2 mm
- board text added: "JCS-BK1091_GO-KART Cockpitplatine Dean 2026 Rev1"
- board text removed: "JCS-BK1091_GO-KART Dean 2026 v1"
